Commit message: Updates

File: Ned.urdf (robot description, URDF)
Before this commit: robot C:/Users/Kolawole/Documents/University Of Hertfordshire/Bsc Computer Science/Robotics/RoboticsFinale!/Robot.urdf, 10 links, 9 joints
Joints:
- joint joint_1: origin xyz=0 0 0.1065 rpy=0 0 0 -> xyz=0 0 0.1065 rpy=0 0 -0.000001
- joint joint_2: origin xyz=0 0 0.065 rpy=0 -1.57 0 -> xyz=0 0 0.065 rpy=-0.000694 -1.57 0.000694
- joint joint_3: origin xyz=0.221 0.012 0 rpy=0 0 0 -> xyz=0.221 0.012 0 rpy=0 0 0.000001
- joint joint_4: origin xyz=0.032 0.042 0 rpy=-1.568653 -1.57 -0.001347 -> xyz=0.032 0.042 0 rpy=-1.568655 -1.57 -0.001346
- joint joint_6: origin xyz=0.0197 0.00925 0 rpy=0 1.57 0 -> xyz=0.0197 0.00925 0 rpy=0.000009 1.57 0.000009
